Commit message: quase B

File: oba.urdf (robot description, URDF)
Before this commit: robot nome_robo, 4 links, 3 joints
Links:
- removed link link2
- removed link link3
- link link1: geometry collision box size=0.7 0.3 0.7; visual box size=0.7 0.3 0.7
- link link_principal: geometry collision sphere radius=1.1; visual sphere radius=1.1
Joints:
- removed joint joint2
- removed joint joint3
- joint joint1: origin xyz=2.0 0 0 -> xyz=0 1.4 1; type fixed -> continuous
